Commit message: add booster training setting

File: source/extensions/isaaclab.humanoid_tasks/isaaclab/humanoid_tasks/assets/urdf/T1_Sim_fixed_arms.urdf (robot description, URDF)
Before this commit: robot V23RobotAsm, 24 links, 23 joints
Joints:
- joint Left_Ankle_Roll: type fixed -> revolute
- joint Right_Ankle_Roll: type fixed -> revolute
